Commit message: launch file added for rviz2&gz

File: src/arduinobot_description/urdf/robot.urdf.xacro (robot description, xacro)
@@ -2,6 +2,13 @@
 <robot xmlns:xacro="http://www.ros.org/wiki/xacro" name="myRobot">
     <!-- <xacro:property name="" value="" /> -->
+    <!-- <xacro:property name="pi" value="3.14159" /> -->
     <xacro:property name="effort" value="30.0" />
     <xacro:property name="velocity" value="10.0" />
+    <xacro:macro name="default_inertia" params="mass">
+        <inertial>
+            <mass value="${mass}"/>
+            <inertia ixx="1" ixy="0.0" ixz="0.0" iyy="1" iyz="0.0" izz="1"/>
+        </inertial>
+    </xacro:macro>
     <!-- ##################################################################################### -->
     <!-- Links -->
@@ -14,4 +21,11 @@
             </geometry>
         </visual>
+        <collision>
+            <origin xyz="-0.5 -0.5 0.0" rpy="0.0 0.0 0.0"/>
+            <geometry>
+                <mesh filename="package://arduinobot_description/meshes/basement.STL" scale="0.01 0.01 0.01"/>
+            </geometry>
+        </collision>
+        <xacro:default_inertia mass="1.0"/>
     </link>
     <link name="base_plate">
@@ -22,4 +36,11 @@
             </geometry>
         </visual>
+        <collision>
+            <origin xyz="-0.39 -0.39 -0.56" rpy="0.0 0.0 0.0"/>
+            <geometry>
+                <mesh filename="package://arduinobot_description/meshes/base_plate.STL" scale="0.01 0.01 0.01"/>
+            </geometry>
+        </collision>
+        <xacro:default_inertia mass="0.1"/>
     </link>
     <link name="forward_drive_arm">
@@ -30,4 +51,11 @@
             </geometry>
         </visual>
+        <collision>
+            <origin xyz="0.19 0.06 -0.08" rpy="0.0 ${-pi/2} ${pi/2}"/>
+            <geometry>
+                <mesh filename="package://arduinobot_description/meshes/forward_drive_arm.STL" scale="0.01 0.01 0.01"/>
+            </geometry>
+        </collision>
+        <xacro:default_inertia mass="0.1"/>
     </link>
     <link name="horizontal_arm">
@@ -38,4 +66,11 @@
             </geometry>
         </visual>
+        <collision>
+            <origin xyz="-0.03 -0.4 -0.06" rpy="${pi/2} 0 ${pi/2}"/>
+            <geometry>
+                <mesh filename="package://arduinobot_description/meshes/horizontal_arm.STL" scale="0.01 0.01 0.01"/>
+            </geometry>
+        </collision>
+        <xacro:default_inertia mass="0.1"/>
     </link>
     <link name="claw_support">
@@ -46,4 +81,11 @@
             </geometry>
         </visual>
+        <collision>
+            <origin xyz="0.0 -0.05 -0.15" rpy="0.0 0.0 ${pi/2}"/>
+            <geometry>
+                <mesh filename="package://arduinobot_description/meshes/claw_support.STL" scale="0.01 0.01 0.01"/>
+            </geometry>
+        </collision>
+        <xacro:default_inertia mass="0.05"/>
     </link>
     <link name="gripper_right">
@@ -54,4 +96,11 @@
             </geometry>
         </visual>
+        <collision>
+            <origin xyz="-0.1 0.5 -0.1" rpy="0 0 ${-pi/2}"/>
+            <geometry>
+                <mesh filename="package://arduinobot_description/meshes/right_finger.STL" scale="0.01 0.01 0.01"/>
+            </geometry>
+        </collision>
+        <xacro:default_inertia mass="0.01"/>
     </link>
     <link name="gripper_left">
@@ -62,4 +111,27 @@
             </geometry>
         </visual>
+        <collision>
+            <origin xyz="-0.04 0.5 -0.1" rpy="0.0 0.0 ${-pi/2}"/>
+            <geometry>
+                <mesh filename="package://arduinobot_description/meshes/left_finger.STL" scale="0.01 0.01 0.01"/>
+            </geometry>
+        </collision>
+        <xacro:default_inertia mass="0.01"/>
+    </link>
+    <link name="rgb_camera">
+        <visual>
+            <!-- <origin xyz="-0.1 -0.14 0.129" rpy="0 ${pi/2} 0.0"/> -->
+            <origin rpy="-1.57 0 -1.57" xyz="-0.1 0.125 0.15"/>
+            <geometry>
+                <mesh filename="package://arduinobot_description/meshes/pi_camera.STL" scale="0.01 0.01 0.01"/>
+            </geometry>
+        </visual>
+        <collision>
+            <origin rpy="-1.57 0 -1.57" xyz="-0.1 0.125 0.15"/>
+            <geometry>
+                <mesh filename="package://arduinobot_description/meshes/pi_camera.STL" scale="0.01 0.01 0.01"/>
+            </geometry>
+        </collision>
+        <xacro:default_inertia mass="0.01"/>
     </link>
     <!-- ##################################################################################### -->
@@ -111,3 +183,8 @@
         <limit lower="0.0" upper="${pi/2}" effort="${effort}" velocity="${velocity}"/>
     </joint>
+    <joint name="base_link_to_rgb_camera" type="fixed">
+        <parent link="base_link"/>
+        <child link="rgb_camera"/>
+        <origin xyz="0.0 0.45 0.2" rpy="0.0 -0.5 ${pi/2}"/>
+    </joint>
 </robot>
